File: elec/layout/default/voltagedivider.kicad_pcb (KiCad board)
At the start: 2 copper layers, 225.7 x 100.8 mm, 0 parts

Commit message: Configure project
Other:
- board text added: "{{GITHASH}}"
- board text removed: "{{"
Changed lines of the file:
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@@
   (gr_line (start 225.62 117.79) (end 257.62 117.79)
     (stroke (width 0.1) (type solid)) (layer "Edge.Cuts"))
-  (gr_text "{{"{{GITHASH}}"}}" (at 152.4 139.7) (layer "F.SilkS")
+  (gr_text "{{GITHASH}}" (at 152.4 139.7) (layer "F.SilkS")
     (effects (font (size 2 2) (thickness 0.1)) (justify left bottom))
   )
-  (gr_text "{{"{{GITHASH}}"}}" (at 62.23 146.05) (layer "F.SilkS")
+  (gr_text "{{GITHASH}}" (at 62.23 146.05) (layer "F.SilkS")
     (effects (font (size 2 2) (thickness 0.1)) (justify left bottom))
   )
-  (gr_text "{{"{{GITHASH}}"}}" (at 232.508427 115.791573) (layer "F.SilkS")
+  (gr_text "{{GITHASH}}" (at 232.508427 115.791573) (layer "F.SilkS")
     (effects (font (size 2 2) (thickness 0.1)) (justify left bottom))
   )
